File: pcb/pegpixel-pcb.brd (EAGLE design)
At the start: 100 x 80 mm, 15 parts

Commit message: add first pcb layout
Parts:
- removed PAD1: 5V IN, wirepad:1,6/0,8
- removed PAD10: SDA OUT, wirepad:1,6/0,8
- removed PAD11: SCL OUT, wirepad:1,6/0,8
- removed PAD12: GND OUT, wirepad:1,6/0,8
- removed PAD2: 3V IN, wirepad:1,6/0,8
- removed PAD3: D IN, wirepad:1,6/0,8
- removed PAD4: SDA IN, wirepad:1,6/0,8
- removed PAD5: SCL IN, wirepad:1,6/0,8
- removed PAD6: GND IN, wirepad:1,6/0,8
- removed PAD7: 5V OUT, wirepad:1,6/0,8
- removed PAD8: 3V OUT, wirepad:1,6/0,8
- removed PAD9: D OUT, wirepad:1,6/0,8
- added D_IN, D_OUT, GND_IN, GND_OUT, SCL_IN, SCL_OUT, SDA_IN, SDA_OUT, VCC_IN, VCC_OUT: WIREPADSMD1,27-254, wirepad:SMD1,27-2,54
- moved C1 45.2 mm to (11.2, 21.3), turned to 180 degrees
- moved LED1 37.0 mm to (10.9, 15.8)
- moved H1 28.1 mm to (11.0, 9.78), turned to 90 degrees
Connections:
- removed net N$1: C1.1, LED1.1-VDD, PAD1.1, PAD7.1
- removed net N$3: C1.2, H1.3, LED1.3-GND, PAD12.1, PAD6.1
- new net GND: C1.2, GND_IN.1, GND_OUT.1, H1.3, LED1.3-GND
- net N$2: now also C1.1, LED1.1-VDD, VCC_IN.1, VCC_OUT.1; no longer PAD2.1, PAD8.1
- net N$4: now also SCL_IN.1, SCL_OUT.1; no longer PAD11.1, PAD5.1
- net N$5: now also SDA_IN.1, SDA_OUT.1; no longer PAD10.1, PAD4.1
- net N$6: now also D_IN.1; no longer PAD3.1
- net N$7: now also D_OUT.1; no longer PAD9.1
Routing:
- net N$2: track 0.00 -> 40.7 mm
- net N$4: track 0.00 -> 27.0 mm, vias 0 -> 3
- net N$5: track 0.00 -> 22.1 mm, vias 0 -> 2
- net N$6: track 0.00 -> 8.29 mm
- net N$7: track 0.00 -> 7.64 mm
- added copper zone on layer 1, net GND
Other:
- board size 100 x 80 mm -> 23.1 x 17.2 mm
