File: pcb-dupont-connectors/pegpixel-pcb.brd (EAGLE design)
At the start: 21.6 x 14.2 mm, 5 parts

Commit message: pcb-design: add missing GRND-via
Parts:
- renumbered C1 to 104
Other:
- board text added: "D"
- board text added: "GND"
- board text added: "PegPixel v1"
- board text added: "SCL"
- board text added: "SDA"
- board text added: "VCC"
- board text removed: "A1454"
- board text removed: "PegPixel"
- board text removed: "SK6812"
Changed lines of the file:
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@@
 <setting verticaltext="up"/>
 </settings>
-<grid distance="0.25" unitdist="mm" unit="mm" style="lines" multiple="5" display="no" altdistance="5" altunitdist="mil" altunit="mil"/>
+<grid distance="0.1" unitdist="mm" unit="mm" style="lines" multiple="5" display="no" altdistance="5" altunitdist="mil" altunit="mil"/>
 <layers>
 <layer number="1" name="Top" color="4" fill="1" visible="yes" active="yes"/>
@@
 </layers>
 <board>
-<fusionsync huburn="a.cGVyc29uYWw6dWUyY2NlYWRm" projecturn="a.cGVyc29uYWw6dWUyY2NlYWRmIzIwMTgxMjA1MTYzOTU0MjU2" f3durn="urn:adsk.wipprod:dm.lineage:qyzXckb4RcSP1Y-8RWG8IQ" pcbguid="1db987de-61c2-4902-8df2-387487b94e24" lastpulledtime="" lastsyncedchangeguid="ca40a10c-09b8-6523-202c-a32f8eccca43"/>
+<fusionsync huburn="a.cGVyc29uYWw6dWUyY2NlYWRm" projecturn="a.cGVyc29uYWw6dWUyY2NlYWRmIzIwMTgxMjA1MTYzOTU0MjU2" f3durn="urn:adsk.wipprod:dm.lineage:qyzXckb4RcSP1Y-8RWG8IQ" pcbguid="1db987de-61c2-4902-8df2-387487b94e24" lastpulledtime="" lastsyncedchangeguid="f528fcf7-35c6-5123-f53d-10015996d344"/>
 <plain>
 <wire x1="0.733446875" y1="14.2170375" x2="0.748859375" y2="0.280228125" width="0" layer="20"/>
@@
 <wire x1="22.368859375" y1="14.226228125" x2="0.978853125" y2="14.227021875" width="0" layer="20"/>
 <wire x1="0.978853125" y1="14.227021875" x2="0.733446875" y2="14.2170375" width="0" layer="20"/>
-<text x="17.998859375" y="2.526228125" size="1.778" layer="25" rot="R90.1">PegPixel</text>
-<text x="7.248859375" y="1.276228125" size="1.016" layer="25" rot="R90">A1454</text>
-<text x="8.498859375" y="4.776228125" size="1.016" layer="25" rot="R90">SK6812</text>
+<text x="17.798859375" y="0.826228125" size="1.778" layer="25" rot="R90.1">PegPixel v1</text>
+<text x="4.95" y="11.7" size="1.016" layer="25">VCC</text>
+<text x="4.95" y="9.15" size="1.016" layer="25">D</text>
+<text x="4.95" y="6.65" size="1.016" layer="25">SDA</text>
+<text x="4.95" y="3.95" size="1.016" layer="25">SCL</text>
+<text x="4.95" y="1.55" size="1.016" layer="25">GND</text>
 </plain>
 <attributes>
@@
 </autorouter>
 <elements>
-<element name="C1" library="rcl" library_urn="urn:adsk.eagle:library:334" package="C0805" package3d_urn="urn:adsk.eagle:package:23617/2" value="104" x="12.208859375" y="12.346228125" smashed="yes">
+<element name="104" library="rcl" library_urn="urn:adsk.eagle:library:334" package="C0805" package3d_urn="urn:adsk.eagle:package:23617/2" value="104" x="12.208859375" y="12.346228125" smashed="yes">
 <attribute name="SPICEPREFIX" value="C" x="42.688859375" y="8.536228125" size="1.778" layer="27" display="off"/>
-<attribute name="VALUE" x="9.438859375" y="10.806228125" size="1.016" layer="27" rot="R90"/>
+<attribute name="VALUE" x="13.438859375" y="11.306228125" size="1.016" layer="25" rot="R180"/>
 </element>
 <element name="H1" library="a1454" package="TSSOP8" package3d_urn="urn:adsk.eagle:package:20813/2" value="A1454SMD" x="11.968859375" y="2.306228125" smashed="yes" rot="R90"/>
@@
 <contactref element="JP1" pad="1"/>
 <contactref element="JP2" pad="1"/>
-<contactref element="C1" pad="1"/>
+<contactref element="104" pad="1"/>
 <wire x1="14.875" y1="1.875" x2="14.875" y2="1.75" width="0.3048" layer="1"/>
 <wire x1="14.875" y1="1.75" x2="14.875" y2="1.375" width="0.3048" layer="1"/>
@@
 <signal name="GND">
 <contactref element="LED1" pad="3-GND"/>
-<contactref element="C1" pad="2"/>
+<contactref element="104" pad="2"/>
 <contactref element="H1" pad="3"/>
 <polygon width="0.1524" layer="1">
@@
 <via x="7.5" y="10.5" extent="1-16" drill="0.35"/>
 <via x="14.75" y="12.75" extent="1-16" drill="0.35"/>
+<via x="17.8" y="8" extent="1-16" drill="0.35"/>
 </signal>
 <signal name="DIN">
